File: GreenCircuit.sch (KiCad schematic (older format))
At the start: 69 parts, among them J1 AVR ISP 6, SW1 SW_Push, SW10 SW_Push, SW11 SW_Push, SW12 SW_Push, SW13 SW_Push, SW14 SW_Push, SW15 SW_Push, SW16 SW_Push, SW17 SW_Push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

Commit message: add indicative LED
Parts:
- R1, R2, R3, R5, R6: footprint Resistor_THT:R_Axial_DIN0204_L3.6mm_D1.6mm_P5.08mm_Horizontal -> Resistor_THT:R_Axial_DIN0207_L6.3mm_D2.5mm_P7.62mm_Horizontal
- renumbered J to J2
Connections:
- net +5V: no longer R6.1
- net at U1.12 (PD6): now also R6.1
- no-connect marks 9 -> 8
Other:
- moved on the sheet: D26, R6
Changed lines of the file:
@@
 F 0 "R5" H 2170 4896 50  0000 L CNN
 F 1 "10kΩ" H 2170 4805 50  0000 L CNN
-F 2 "Resistor_THT:R_Axial_DIN0204_L3.6mm_D1.6mm_P5.08mm_Horizontal" V 2030 4850 50  0001 C CNN
+F 2 "Resistor_THT:R_Axial_DIN0207_L6.3mm_D2.5mm_P7.62mm_Horizontal" V 2030 4850 50  0001 C CNN
 F 3 "~" H 2100 4850 50  0001 C CNN
 	1    2100 4850
@@
 Row2
 $Comp
-L power:+5V #PWR09
-U 1 1 5F180EA9
-P 1600 3650
-F 0 "#PWR09" H 1600 3500 50  0001 C CNN
-F 1 "+5V" H 1615 3823 50  0000 C CNN
-F 2 "" H 1600 3650 50  0001 C CNN
-F 3 "" H 1600 3650 50  0001 C CNN
-	1    1600 3650
-	1    0    0    -1
-$EndComp
-$Comp
 L power:GND #PWR012
 U 1 1 5F1815E7
-P 2800 3950
-F 0 "#PWR012" H 2800 3700 50  0001 C CNN
-F 1 "GND" H 2805 3777 50  0000 C CNN
-F 2 "" H 2800 3950 50  0001 C CNN
-F 3 "" H 2800 3950 50  0001 C CNN
-	1    2800 3950
+P 6500 5300
+F 0 "#PWR012" H 6500 5050 50  0001 C CNN
+F 1 "GND" H 6505 5127 50  0000 C CNN
+F 2 "" H 6500 5300 50  0001 C CNN
+F 3 "" H 6500 5300 50  0001 C CNN
+	1    6500 5300
 	1    0    0    -1
 $EndComp
@@
 L Device:LED D26
 U 1 1 5F181E2F
-P 2400 3900
-F 0 "D26" H 2393 3645 50  0000 C CNN
-F 1 "LED" H 2393 3736 50  0000 C CNN
-F 2 "LED_THT:LED_D3.0mm" H 2400 3900 50  0001 C CNN
-F 3 "~" H 2400 3900 50  0001 C CNN
-	1    2400 3900
+P 6250 4800
+F 0 "D26" H 6243 4545 50  0000 C CNN
+F 1 "LED" H 6243 4636 50  0000 C CNN
+F 2 "LED_THT:LED_D3.0mm" H 6250 4800 50  0001 C CNN
+F 3 "~" H 6250 4800 50  0001 C CNN
+	1    6250 4800
 	-1   0    0    1
 $EndComp
@@
 L Device:R R6
 U 1 1 5F187FA3
-P 1900 3900
-F 0 "R6" V 2107 3900 50  0000 C CNN
-F 1 "1.5kΩ" V 2016 3900 50  0000 C CNN
-F 2 "Resistor_THT:R_Axial_DIN0204_L3.6mm_D1.6mm_P5.08mm_Horizontal" V 1830 3900 50  0001 C CNN
-F 3 "~" H 1900 3900 50  0001 C CNN
-	1    1900 3900
-	0    -1   -1   0
-$EndComp
-Wire Wire Line
-	1600 3650 1600 3900
-Wire Wire Line
-	1600 3900 1750 3900
-Wire Wire Line
-	2050 3900 2250 3900
-Wire Wire Line
-	2550 3900 2800 3900
-Wire Wire Line
-	2800 3900 2800 3950
+P 5800 4800
+F 0 "R6" V 6007 4800 50  0000 C CNN
+F 1 "1.5kΩ" V 5916 4800 50  0000 C CNN
+F 2 "Resistor_THT:R_Axial_DIN0207_L6.3mm_D2.5mm_P7.62mm_Horizontal" V 5730 4800 50  0001 C CNN
+F 3 "~" H 5800 4800 50  0001 C CNN
+	1    5800 4800
+	0    -1   -1   0
+$EndComp
+Wire Wire Line
+	5950 4800 6100 4800
+Wire Wire Line
+	6400 4800 6500 4800
+Wire Wire Line
+	6500 4800 6500 5300
 Text GLabel 5450 3400 2    50   Input ~ 0
 Row0
@@
 NoConn ~ 5450 3900
 $Comp
-L Connector:USB_A J
+L Connector:USB_A J2
 U 1 1 5F46B763
 P 1550 1950
-F 0 "J" H 1607 2417 50  0000 C CNN
+F 0 "J2" H 1607 2417 50  0000 C CNN
 F 1 "USB_A-Connector" H 1607 2326 50  0000 C CNN
 F 2 "Connector_USB:USB_A_CONNFLY_DS1095-WNR0" H 1700 1900 50  0001 C CNN
@@
 F 0 "R1" V 2943 1950 50  0000 C CNN
 F 1 "75Ω" V 3034 1950 50  0000 C CNN
-F 2 "Resistor_THT:R_Axial_DIN0204_L3.6mm_D1.6mm_P5.08mm_Horizontal" V 3080 1950 50  0001 C CNN
+F 2 "Resistor_THT:R_Axial_DIN0207_L6.3mm_D2.5mm_P7.62mm_Horizontal" V 3080 1950 50  0001 C CNN
 F 3 "~" H 3150 1950 50  0001 C CNN
 	1    3150 1950
@@
 F 0 "R2" V 2943 2050 50  0000 C CNN
 F 1 "75Ω" V 3034 2050 50  0000 C CNN
-F 2 "Resistor_THT:R_Axial_DIN0204_L3.6mm_D1.6mm_P5.08mm_Horizontal" V 3080 2050 50  0001 C CNN
+F 2 "Resistor_THT:R_Axial_DIN0207_L6.3mm_D2.5mm_P7.62mm_Horizontal" V 3080 2050 50  0001 C CNN
 F 3 "~" H 3150 2050 50  0001 C CNN
 	1    3150 2050
@@
 F 0 "R3" H 2820 1646 50  0000 L CNN
 F 1 "1.5kΩ" H 2820 1555 50  0000 L CNN
-F 2 "Resistor_THT:R_Axial_DIN0204_L3.6mm_D1.6mm_P5.08mm_Horizontal" V 2680 1600 50  0001 C CNN
+F 2 "Resistor_THT:R_Axial_DIN0207_L6.3mm_D2.5mm_P7.62mm_Horizontal" V 2680 1600 50  0001 C CNN
 F 3 "~" H 2750 1600 50  0001 C CNN
 	1    2750 1600
@@
 NoConn ~ 5450 4300
 NoConn ~ 5450 4600
-NoConn ~ 5450 4800
 $Comp
 L Mechanical:MountingHole H1
@@
 Wire Wire Line
 	1850 2050 2450 2050
+Wire Wire Line
+	5450 4800 5650 4800
 $EndSCHEMATC

Commit message: 220ohm for LED
Parts:
- R6: value 1.5kΩ -> 220Ω
Changed lines of the file:
@@
 P 5800 4800
 F 0 "R6" V 6007 4800 50  0000 C CNN
-F 1 "1.5kΩ" V 5916 4800 50  0000 C CNN
+F 1 "220Ω" V 5916 4800 50  0000 C CNN
 F 2 "Resistor_THT:R_Axial_DIN0207_L6.3mm_D2.5mm_P7.62mm_Horizontal" V 5730 4800 50  0001 C CNN
 F 3 "~" H 5800 4800 50  0001 C CNN

Commit message: v0.5
Parts:
- removed J2: USB_A-Connector, Connector_USB:USB_A_CONNFLY_DS1095-WNR0, symbol Connector:USB_A
- added J1: USB_B_Mini, digikey-footprints:USB_Mini_B_Female_548190519, symbol Connector:USB_B_Mini
- renumbered J1 to J2
Connections:
- net D-: now also U1.3 (PD1); no longer U1.5 (PD3)
- net DN: now also J1.2 (D-)
- net DP: now also J1.3 (D+)
- net GND: now also J1.5 (GND), J1.6 (Shield)
- net at F1.2: now also J1.1 (VBUS)
- no-connect marks 8 -> 9
Other:
- moved on the sheet: C1, C2, C3, C4, C5, D24, D25, D26, F1, J2, R1, R2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

Commit message: new pcb size with M3 screw for buttom acrylic
Parts:
- H1, H2, H3, H4: footprint MountingHole:MountingHole_2.2mm_M2 -> MountingHole:MountingHole_3.2mm_M3
Changed lines of the file:
@@
 F 0 "H1" H 9450 5846 50  0000 L CNN
 F 1 "MountingHole" H 9450 5755 50  0001 L CNN
-F 2 "MountingHole:MountingHole_2.2mm_M2" H 9350 5800 50  0001 C CNN
+F 2 "MountingHole:MountingHole_3.2mm_M3" H 9350 5800 50  0001 C CNN
 F 3 "~" H 9350 5800 50  0001 C CNN
 	1    9350 5800
@@
 F 0 "H2" H 9750 5846 50  0000 L CNN
 F 1 "MountingHole" H 9750 5755 50  0001 L CNN
-F 2 "MountingHole:MountingHole_2.2mm_M2" H 9650 5800 50  0001 C CNN
+F 2 "MountingHole:MountingHole_3.2mm_M3" H 9650 5800 50  0001 C CNN
 F 3 "~" H 9650 5800 50  0001 C CNN
 	1    9650 5800
@@
 F 0 "H3" H 9450 6046 50  0000 L CNN
 F 1 "MountingHole" H 9450 5955 50  0001 L CNN
-F 2 "MountingHole:MountingHole_2.2mm_M2" H 9350 6000 50  0001 C CNN
+F 2 "MountingHole:MountingHole_3.2mm_M3" H 9350 6000 50  0001 C CNN
 F 3 "~" H 9350 6000 50  0001 C CNN
 	1    9350 6000
@@
 F 0 "H4" H 9750 6046 50  0000 L CNN
 F 1 "MountingHole" H 9750 5955 50  0001 L CNN
-F 2 "MountingHole:MountingHole_2.2mm_M2" H 9650 6000 50  0001 C CNN
+F 2 "MountingHole:MountingHole_3.2mm_M3" H 9650 6000 50  0001 C CNN
 F 3 "~" H 9650 6000 50  0001 C CNN
 	1    9650 6000
@@
 F 3 "http://ww1.microchip.com/downloads/en/DeviceDoc/ATmega328_P%20AVR%20MCU%20with%20picoPower%20Technology%20Data%20Sheet%2040001984A.pdf" H 4700 4150 50  0001 C CNN
 	1    4700 4150
-	1    0    0    -1
-$EndComp
-$Comp
-L Graphic:Logo_Open_Hardware_Large #LOGO1
-U 1 1 5F56A161
-P 10500 5900
-F 0 "#LOGO1" H 10500 6400 50  0001 C CNN
-F 1 "Logo_Open_Hardware_Large" H 10500 5500 50  0001 C CNN
-F 2 "" H 10500 5900 50  0001 C CNN
-F 3 "~" H 10500 5900 50  0001 C CNN
-	1    10500 5900
 	1    0    0    -1
 $EndComp
@@
 Wire Wire Line
 	1550 2800 2150 2800
-NoConn ~ 5300 4950
 Wire Wire Line
 	8850 1350 8850 1650
@@
 	0    -1   -1   0
 $EndComp
+$Comp
+L Graphic:Logo_Open_Hardware_Small #LOGO1
+U 1 1 5F9B5001
+P 10500 5800
+F 0 "#LOGO1" H 10500 6075 50  0001 C CNN
+F 1 "Logo_Open_Hardware_Small" H 10500 5575 50  0001 C CNN
+F 2 "Symbol:KiCad-Logo_8mm_Copper" H 10500 5800 50  0001 C CNN
+F 3 "~" H 10500 5800 50  0001 C CNN
+	1    10500 5800
+	1    0    0    -1
+$EndComp
+$Comp
+L Graphic:Logo_Open_Hardware_Small #LOGO2
+U 1 1 5F9B59EC
+P 10150 6150
+F 0 "#LOGO2" H 10150 6425 50  0001 C CNN
+F 1 "Logo_Open_Hardware_Small" H 10150 5925 50  0001 C CNN
+F 2 "Symbol:OSHW-Logo2_7.3x6mm_Copper" H 10150 6150 50  0001 C CNN
+F 3 "~" H 10150 6150 50  0001 C CNN
+	1    10150 6150
+	1    0    0    -1
+$EndComp
+NoConn ~ 5300 4950
 $EndSCHEMATC
